File: sch/nRF54L15.kicad_sch (KiCad schematic)
At the start: 43 parts, among them J7 Conn_01x05_MountingPin, SW2 SW_Push, U1 nRF54L15-QFAA, U11 SHT4x, U12 ADXL367, U13 ZD25WQ16CEIGR, U9 STEMMA-QT, X1 32MHz, X2 32.768kHz

Commit message: Updates for rev 1
Parts:
- added D1: LED_Blue, LED_SMD:LED_0603_1608Metric, symbol Device:LED_Small
- added R13: 1kR, passives:C_0201_0603Metric_L, symbol Device:R_Small_US
- added TP14, TP15, TP16, TP17, TP18, TP19, TP20, TP21, TP22, TP23: TestPoint, TestPoint:TestPoint_Pad_D1.0mm, symbol Connector:TestPoint
- AE1: LCSC (none) -> C89334
- C1, C2, C3, C4, C54, C55, C57, C58: LCSC (none) -> C76935
- C10, C7: LCSC (none) -> C319184
- C11: LCSC (none) -> C161289
- C12: LCSC (none) -> C5142551
- C13: LCSC (none) -> C80433
- C5: LCSC (none) -> C15525
- C52, C53: value C_Small -> 300pF; LCSC (none) -> C2180639
- C56: LCSC (none) -> C76932
- C6: LCSC (none) -> C161414
- C8: LCSC (none) -> C76926
- C9: LCSC (none) -> C161419
- FB1: LCSC (none) -> C97850
- J7: LCSC (none) -> C5337029
- L1: LCSC (none) -> C48944999
- L2: LCSC (none) -> C7216765
- L3, L4: LCSC (none) -> C3911055
- R1: LCSC (none) -> C138165
- R10, R11, R12, R9: LCSC (none) -> C270344
- SW2: LCSC (none) -> C127488
- U1: LCSC (none) -> C42458750
- U11: LCSC (none) -> C2848306
- U12: LCSC (none) -> C17643415
- U9: LCSC (none) -> C160404
- X1: LCSC (none) -> C383840
- X2: LCSC (none) -> C99009
- Z5: LCSC (none) -> C473473
Connections:
- net GND: now also R13.2
- net INT1: now also TP23.1
- net RX: now also TP15.1
- net SCL_SENSOR: now also TP21.1
- net SCL_STEMMA: now also TP22.1
- net SDA_SENSOR: now also TP19.1
- net SDA_STEMMA: now also TP20.1
- net SWDCLK: now also TP17.1
- net SWDIO: now also TP16.1
- net TX: now also TP14.1
- net ~{RESET}: now also TP18.1
- net at U1.8 (P1.07): now also D1.2 (A)
- new net: D1.1 (K), R13.1
- no-connect marks 6 -> 5

Commit message: Updates
Parts:
- D1: LCSC C965807 -> C7496819
- U12: footprint amemb-Package_LGA:amemb-ADXL367_LGA-12_2.11x2.21mm_P0.5mm_LayoutBorder2x4y -> easyeda2kicad:ADXL367_LGA-12_2.11x2.21mm_P0.5mm_LayoutBorder2x4y; symbol amemb-Sensor_Motion:ADXL367 -> easyeda2kicad:ADXL367
- U9: footprint amemb-Conenctor_JST:JST_SH_SM04B-SRSS-TB_1x04-1MP_P1.00mm_Horizontal -> easyeda2kicad:JST_SH_SM04B-SRSS-TB_1x04-1MP_P1.00mm_Horizontal; symbol amemb-Connector:STEMMA-QT -> easyeda2kicad:STEMMA-QT
Changed lines of the file:
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@@
 	)
 	(symbol
-		(lib_id "amemb-Connector:STEMMA-QT")
+		(lib_id "easyeda2kicad:STEMMA-QT")
 		(at 52.07 58.42 0)
 		(unit 1)
@@
 			)
 		)
-		(property "Footprint" "amemb-Conenctor_JST:JST_SH_SM04B-SRSS-TB_1x04-1MP_P1.00mm_Horizontal"
+		(property "Footprint" "easyeda2kicad:JST_SH_SM04B-SRSS-TB_1x04-1MP_P1.00mm_Horizontal"
 			(at 52.07 58.42 0)
 			(hide yes)
@@
 	)
 	(symbol
-		(lib_id "amemb-Sensor_Motion:ADXL367")
+		(lib_id "easyeda2kicad:ADXL367")
 		(at -62.23 198.12 0)
 		(mirror y)
@@
 			)
 		)
-		(property "Footprint" "amemb-Package_LGA:amemb-ADXL367_LGA-12_2.11x2.21mm_P0.5mm_LayoutBorder2x4y"
+		(property "Footprint" "easyeda2kicad:ADXL367_LGA-12_2.11x2.21mm_P0.5mm_LayoutBorder2x4y"
 			(at -62.23 198.12 0)
 			(hide yes)
@@
 			)
 		)
-		(property "LCSC" "C965807"
+		(property "LCSC" "C7496819"
 			(at 115.57 102.87 90)
 			(hide yes)
