File: sch/nRF54L15.kicad_sch (KiCad schematic)
At the start: 55 parts, among them J7 Conn_01x05_MountingPin, SW2 SW_Push, U1 nRF54L15-QFAA, U11 SHT4x, U12 ADXL367, U13 ZD25WQ16CEIGR, U9 STEMMA-QT, X1 32MHz, X2 32.768kHz

Commit message: Revision 0.2
Parts:
- removed C56: 220nF, passives:C_0201_0603Metric_L, symbol Device:C_Small
- removed U12: ADXL367, easyeda2kicad:ADXL367_LGA-12_2.11x2.21mm_P0.5mm_LayoutBorder2x4y, symbol easyeda2kicad:ADXL367
- added U18: LIS2DH, Package_LGA:LGA-14_2x2mm_P0.35mm_LayoutBorder3x4y, symbol Sensor_Motion:LIS2DH
- C52, C53: value 300pF -> 330pF; LCSC C2180639 -> C237559
- U13: value ZD25WQ16CEIGR -> W25Q16JVUXIQ; LCSC C7304007 -> C2843335
Connections:
- net GND: now also U18.10 (GND), U18.11 (GND), U18.12 (GND), U18.13 (GND), U18.14 (GND), U18.9 (GND)
- net INT1: now also U18.6 (INT1)
- net SCL_SENSOR: now also U18.1 (SCL/SPC)
- net SDA_SENSOR: now also U18.2 (SDA/SDI)
- net SENSOR_VDD: now also U18.3 (SDO), U18.4 (~{CS}), U18.7 (Vdd_IO), U18.8 (Vdd)
- net at Z5.2, Z6.2: now also AE1.1 (FEED); no longer AE1.2 (PCB_Trace)
- no-connect marks 5 -> 4
Other:
- moved on the sheet: AE1, C54, C55, C57, C58, R11, R12, U11, U13

Commit message: Updates for V2
Parts:
- U13: value W25Q16JVUXIQ -> MX25R1635FZUIL0; LCSC C2843335 -> C152595
- X1: value 32MHz -> 32MHz, 10pF; LCSC C383840 -> C54427949
Changed lines of the file:
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@@
 			)
 		)
-		(property "Value" "W25Q16JVUXIQ"
+		(property "Value" "MX25R1635FZUIL0"
 			(at 76.2 177.7999 0)
 			(show_name no)
@@
 			)
 		)
-		(property "Datasheet" "http://www.winbond.com/resource-files/w25q32jv%20revg%2003272018%20plus.pdf"
+		(property "Datasheet" "https://www.macronix.com/Lists/Datasheet/Attachments/8702/MX25R1635F%2C%20Wide%20Range%2C%2016Mb%2C%20v1.6.pdf"
 			(at 87.63 179.07 0)
 			(hide yes)
@@
 			)
 		)
-		(property "Description" "32Mbit / 4MiB Serial Flash Memory, Standard/Dual/Quad SPI, 2.7-3.6V, WSON-8"
+		(property "Description" "16Mbit / 2MiB Ultra Low Power Serial NOR Flash Memory, Standard/Dual/Quad SPI, 1.65-3.6V, 33MHz"
 			(at 87.63 176.53 0)
 			(hide yes)
@@
 			)
 		)
-		(property "LCSC" "C2843335"
+		(property "LCSC" "C152595"
 			(at 87.63 176.53 0)
 			(hide yes)
@@
 			)
 		)
-		(property "Value" "32MHz"
+		(property "Value" "32MHz, 10pF"
 			(at 115.57 53.34 0)
 			(show_name no)
@@
 			)
 		)
-		(property "Datasheet" ""
+		(property "Datasheet" "https://atta.szlcsc.com/upload/public/pdf/source/20260323/688CCC4499BA77041AC465C19328DD85.pdf"
 			(at 119.38 52.07 0)
 			(hide yes)
@@
 			)
 		)
-		(property "Description" ""
+		(property "Description" "32MHz crystal, 10pF, 40 ohm ESR max, C0 <= 3pF, 2.0x1.6mm 4-pad SMD; pins 2 and 4 grounded"
 			(at 119.38 52.07 0)
 			(show_name no)
@@
 			)
 		)
-		(property "LCSC" "C383840"
+		(property "LCSC" "C54427949"
 			(at 119.38 52.07 0)
 			(hide yes)
