File: sch/SX1262.kicad_sch (KiCad schematic)
At the start: 20 parts, among them J2 Conn_Coaxial_Small, U3 SX1262IMLTRT, U4 BGS12WN6E6327, Y1 32MHz, 10pF

Commit message: Updates for rev 1
Parts:
- added C59: 1uF, passives:C_0201_0603Metric_L, symbol Device:C_Small
- added TP24, TP25, TP26, TP27, TP28, TP29, TP30, TP31: TestPoint, TestPoint:TestPoint_Pad_D1.0mm, symbol Connector:TestPoint
- C27, C28: LCSC (none) -> C76935
- C29: LCSC (none) -> C88917
- C30: value 47nF -> 470nF; LCSC (none) -> C85926
- C31: LCSC (none) -> C62546
- C32, C34: LCSC (none) -> C66942
- C33: LCSC (none) -> C85904
- FL1: LCSC (none) -> C5224443; now not fitted; now left out of the parts list
- J2: LCSC (none) -> C88374
- L7: LCSC (none) -> C1857885
- L8: LCSC (none) -> C2838019
- R4, R5: LCSC (none) -> C77623
- U3: LCSC (none) -> C191341
- U4: LCSC (none) -> C1854968
- Y1: LCSC (none) -> C383840
- Z2: LCSC (none) -> C473473
Connections:
- net ANT_SW: now also U3.6 (DIO3), TP28.1
- net CLK: now also TP24.1
- net DIO1: now also TP29.1
- net DIO2: now also TP30.1
- net GND: now also C59.2
- net MISO: now also TP25.1
- net MOSI: now also TP26.1
- net VDD_SX1262: now also C59.1; no longer C28.1, C30.1, L8.1, U3.11 (VBAT_IO), U3.7 (VREG)
- net ~{CS}: now also TP27.1
- net ~{RESET}: now also TP31.1
- new net: C30.1, L8.1, U3.7 (VREG)
- new net VDD_nRF: C28.1, U3.11 (VBAT_IO)
- no-connect marks 1 -> 0
Other:
- moved on the sheet: C27

Commit message: Add missing 3D models
Parts:
- FL1: now fitted; now in the parts list
Changed lines of the file:
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@@
 		(body_style 1)
 		(exclude_from_sim no)
-		(in_bom no)
+		(in_bom yes)
 		(on_board yes)
-		(in_pos_files no)
-		(dnp yes)
+		(in_pos_files yes)
+		(dnp no)
 		(fields_autoplaced yes)
 		(property "Reference" "FL1"
