File: sch/SX1262.kicad_sch (KiCad schematic)
At the start: 29 parts, among them J2 Conn_Coaxial_Small, U3 SX1262IMLTRT, U4 BGS12WN6E6327, Y1 32MHz, 10pF

Commit message: Revision 0.2
Parts:
- U4: value BGS12WN6E6327 -> BGS12SN6E6327XTSA1; LCSC C1854968 -> C114953
Changed lines of the file:
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@@
 			)
 		)
-		(property "Value" "BGS12WN6E6327"
+		(property "Value" "BGS12SN6E6327XTSA1"
 			(at 192.3481 95.25 0)
 			(show_name no)
@@
 			)
 		)
-		(property "LCSC" "C1854968"
+		(property "LCSC" " C114953"
 			(at 189.23 107.95 0)
 			(hide yes)

Commit message: Updates for V2
Parts:
- FL1: LCSC C5224443 -> C7434807
- Y1: LCSC C383840 -> C1986260
Changed lines of the file:
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@@
 			)
 		)
-		(property "Datasheet" ""
+		(property "Datasheet" "https://datasheet.lcsc.com/datasheet/pdf/0f4a170f8b3efa2349190a8115e046dc.pdf?productCode=C1986260"
 			(at 72.39 91.44 0)
 			(hide yes)
@@
 			)
 		)
-		(property "Description" "Four pin crystal, GND on pins 2 and 4, small symbol"
+		(property "Description" "32MHz crystal, 10pF, 50 ohm ESR max, C0 <= 0.78pF, 2.0x1.6mm 4-pad SMD; pins 2 and 4 grounded"
 			(at 72.39 91.44 0)
 			(hide yes)
@@
 			)
 		)
-		(property "LCSC" "C383840"
+		(property "LCSC" "C1986260"
 			(at 72.39 91.44 0)
 			(hide yes)
@@
 			)
 		)
-		(property "LCSC" "C5224443"
+		(property "LCSC" "C7434807"
 			(at 156.21 106.68 0)
 			(hide yes)
