File: sch/Debugger.kicad_sch (KiCad schematic)
At the start: 31 parts, among them J3 Conn_ARM_SWD_TagConnect_TC203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, Q1 Q_NMOS_GSD, U10 TPS22991, U6 TXU0204RUTR, U7 nRF52833-QDXX, U8 TXU0101DRYR, Y2 32MHz, 10pF

Commit message: Revision 0.2
Parts:
- added C56: 1uF, passives:C_0201_0603Metric_L, symbol Device:C_Small
- added U12: TMUX1511RSVR, easyeda2kicad:UTQFN-16_L2.6-W1.8-P0.40-BL, symbol easyeda2kicad:TMUX1511RSVR
Connections:
- net GND: now also C56.2, U12.8 (GND)
- net LEVEL_SHIFT_VDD: now also C56.1, U12.1 (SEL1), U12.11 (SEL3), U12.15 (SEL4), U12.16 (VDD), U12.4 (SEL2)
- net RX: now also U12.5 (S2); no longer U6.9 (B2Y)
- net TARGET_SWDCLK: now also U12.2 (S1); no longer U6.10 (B1Y)
- net TARGET_SWDIO: now also U12.14 (S4); no longer U6.7 (B4), U8.4 (BY)
- net TX: now also U12.10 (S3); no longer U6.8 (B3)
- new net INT_TRG.RX: U12.6 (D2), U6.9 (B2Y)
- new net INT_TRG.SWDCLK: U12.3 (D1), U6.10 (B1Y)
- new net INT_TRG.SWDIO: U12.13 (D4), U6.7 (B4), U8.4 (BY)
- new net INT_TRG.TX: U12.9 (D3), U6.8 (B3)

Commit message: Updates for V2
Parts:
- Y2: LCSC C383840 -> C54427949
Other:
- moved on the sheet: C35, C36, C37, C38, C39, C40, C41, C42, C43, C44, C45, C46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
