File: Sidewalk_Devkit.kicad_pcb (KiCad board)
At the start: 6 copper layers, 55 x 34 mm, 117 parts, among them J1 USB_C_Receptacle_USB2.0_16P, J2 Conn_Coaxial_Small, J3 Conn_ARM_SWD_TagConnect_TC203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, J4 Conn_01x02_MountingPin, J7 Conn_01x05_MountingPin, Q1 Q_NMOS_GSD, SW1 SW_Push, SW2 SW_Push, U1 nRF54L15-QFAA, U10 TPS22991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

Commit message: Updates for rev 1
Parts:
- added C59: 1uF, passives:C_0201_0603Metric_L, F.Cu at (134.4, 62.9)
- added D1: LED_Blue, LED_SMD:LED_0603_1608Metric, F.Cu at (132.2, 68.3)
- added D2: LED_Red, LED_SMD:LED_0603_1608Metric, F.Cu at (114.5, 57.2)
- added D3: LED_Green, LED_SMD:LED_0603_1608Metric, F.Cu at (114.5, 58.8)
- added D4: LED_Blue, LED_SMD:LED_0603_1608Metric, F.Cu at (114.5, 60.4)
- added D5: LED_Blue, LED_SMD:LED_0603_1608Metric, F.Cu at (119.0, 75.2)
- added R13: 1kR, passives:C_0201_0603Metric_L, F.Cu at (131.0, 68.7)
- added R17: 1kR, passives:C_0201_0603Metric_L, F.Cu at (120.1, 76.4)
- added TP1: TestPoint, TestPoint:TestPoint_Keystone_5015_Micro_Mini, B.Cu at (102.2, 66.6)
- added TP10: TestPoint, TestPoint:TestPoint_Pad_D1.0mm, B.Cu at (106.0, 56.6)
- added TP11: TestPoint, TestPoint:TestPoint_Pad_D1.0mm, B.Cu at (133.8, 56.0)
- added TP12: TestPoint, TestPoint:TestPoint_Pad_D1.0mm, B.Cu at (136.9, 54.7)
- added TP13: TestPoint, TestPoint:TestPoint_Pad_D1.0mm, B.Cu at (128.2, 55.1)
- added TP14: TestPoint, TestPoint:TestPoint_Pad_D1.0mm, B.Cu at (137.8, 79.2)
- added TP15: TestPoint, TestPoint:TestPoint_Pad_D1.0mm, B.Cu at (137.8, 81.2)
- added TP16: TestPoint, TestPoint:TestPoint_Pad_D1.0mm, B.Cu at (142.5, 81.4)
- added TP17: TestPoint, TestPoint:TestPoint_Pad_D1.0mm, B.Cu at (142.9, 78.3)
- added TP18: TestPoint, TestPoint:TestPoint_Pad_D1.0mm, B.Cu at (105.0, 75.3)
- added TP19: TestPoint, TestPoint:TestPoint_Pad_D1.0mm, B.Cu at (134.4, 75.8)
- added TP2: TestPoint, TestPoint:TestPoint_Pad_D1.0mm, B.Cu at (104.3, 60.3)
- added TP20: TestPoint, TestPoint:TestPoint_Pad_D1.0mm, B.Cu at (110.4, 58.8)
- added TP21: TestPoint, TestPoint:TestPoint_Pad_D1.0mm, B.Cu at (131.8, 73.9)
- added TP22: TestPoint, TestPoint:TestPoint_Pad_D1.0mm, B.Cu at (107.7, 60.4)
- added TP23: TestPoint, TestPoint:TestPoint_Pad_D1.0mm, B.Cu at (127.2, 75.9)
- added TP24: TestPoint, TestPoint:TestPoint_Pad_D1.0mm, B.Cu at (137.5, 77.1)
- added TP25: TestPoint, TestPoint:TestPoint_Pad_D1.0mm, B.Cu at (139.5, 77.4)
- added TP26: TestPoint, TestPoint:TestPoint_Pad_D1.0mm, B.Cu at (145.2, 67.9)
- added TP27: TestPoint, TestPoint:TestPoint_Pad_D1.0mm, B.Cu at (142.6, 76.1)
- added TP28: TestPoint, TestPoint:TestPoint_Pad_D1.0mm, B.Cu at (139.1, 57.7)
- added TP29: TestPoint, TestPoint:TestPoint_Pad_D1.0mm, B.Cu at (143.3, 67.2)
- added TP3: TestPoint, TestPoint:TestPoint_Pad_D1.0mm, B.Cu at (118.8, 54.1)
- added TP30: TestPoint, TestPoint:TestPoint_Pad_D1.0mm, B.Cu at (134.3, 65.1)
- added TP31: TestPoint, TestPoint:TestPoint_Pad_D1.0mm, B.Cu at (136.4, 66.8)
- added TP32: TestPoint, TestPoint:TestPoint_Pad_D1.0mm, B.Cu at (118.3, 68.3)
- added TP33: TestPoint, TestPoint:TestPoint_Pad_D1.0mm, B.Cu at (129.7, 69.3)
- added TP34: TestPoint, TestPoint:TestPoint_Pad_D1.0mm, B.Cu at (127.7, 68.8)
- added TP35: TestPoint, TestPoint:TestPoint_Pad_D1.0mm, B.Cu at (145.4, 79.7)
- added TP4: TestPoint, TestPoint:TestPoint_Pad_D1.0mm, B.Cu at (113.1, 62.1)
- added TP5: TestPoint, TestPoint:TestPoint_Pad_D1.0mm, B.Cu at (114.0, 55.2)
- added TP6: TestPoint, TestPoint:TestPoint_Pad_D1.0mm, B.Cu at (116.1, 65.0)
- added TP7: TestPoint, TestPoint:TestPoint_Pad_D1.0mm, B.Cu at (126.3, 56.1)
- added TP8: TestPoint, TestPoint:TestPoint_Pad_D1.0mm, B.Cu at (132.1, 57.6)
- added TP9: TestPoint, TestPoint:TestPoint_Pad_D1.0mm, B.Cu at (131.3, 65.2)
- C30: value 47nF -> 470nF
- C52, C53: value C_Small -> 300pF
- moved C28 7.90 mm to (134.4, 63.4), turned to 180 degrees
- moved C27 5.88 mm to (140.9, 58.9), turned to 0 degrees
- moved C30 2.09 mm to (135.5, 61.1)
Connections:
- net Net-(U2-PVDD) renamed /nPM1300/VSYS
- C28 pad 1: VDD_SX1262 -> VDD_nRF
- C30 pad 1: VDD_SX1262 -> Net-(U3-VREG)
- L8 pad 1: VDD_SX1262 -> Net-(U3-VREG)
- U1 pad 8: unconnected-(U1-P1.07-Pad8) -> Net-(D1-A)
- U2 pad 18: /nPM1300/NTC -> GND
- U2 pad 25: unconnected-(U2-LED0-Pad25) -> /nPM1300/LED0
- U2 pad 26: unconnected-(U2-LED1-Pad26) -> /nPM1300/LED1
- U2 pad 27: unconnected-(U2-LED2-Pad27) -> /nPM1300/LED2
- U3 pad 11: VDD_SX1262 -> VDD_nRF
- U3 pad 6: unconnected-(U3-DIO3-Pad6) -> /SX1262/ANT_SW
- U3 pad 7: VDD_SX1262 -> Net-(U3-VREG)
- U7 pad 22: unconnected-(U7-P0.09-Pad22) -> Net-(D5-A)
Routing:
- net /SX1262/ANT_SW: track 0.00 -> 17.3 mm, vias 0 -> 2
- net /nPM1300/LED2: track 0.00 -> 15.1 mm, vias 0 -> 2
- net /nPM1300/LED1: track 0.00 -> 14.1 mm, vias 0 -> 2
- net /nPM1300/VSYS: track 1.15 -> 13.7 mm, vias 5 -> 6
- net /nPM1300/LED0: track 0.00 -> 11.2 mm, vias 0 -> 2
- net Net-(D1-A): track 0.00 -> 10.8 mm, vias 0 -> 2
- net /Debugger/DBG_~{RESET}: track 44.3 -> 49.1 mm, vias 2 -> 3
- net /nPM1300/SCL: track 41.6 -> 45.8 mm
- net /Debugger/VBUS: track 9.81 -> 14.0 mm, vias 0 -> 1
- net VDD_nRF: track 73.2 -> 77.4 mm
- net /SX1262/MOSI: track 28.1 -> 32.0 mm
- net /Debugger/RX: track 33.3 -> 37.1 mm, vias 2 -> 3
- net /nRF54L15/SCL_STEMMA: track 59.8 -> 63.3 mm
- net Net-(D5-A): track 0.00 -> 3.40 mm
- net /nRF54L15/SDA_STEMMA: track 59.2 -> 62.4 mm
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Other:
- board text added: "BAT"
- board text added: "BTN"
- board text added: "DEBUGGER"
- board text added: "NFC"
- board text added: "Nordic Semiconductor nRF54L15 + nPM1300 Sidewalk Devkit"
- board text added: "Rev: ${REVISION} @{vcsidentifier(8)} @{vcsdirtysuffix()}"
- board text added: "STEMMA"
- board text added: "SX1262"
- board text added: "nPM1300"
- board text added: "nRF54L15"
- board text added: "~{RST}"

Commit message: Updates
Parts:
- J1: footprint amemb-Connector_USB:USB_C_Receptacle_HRO_TYPE-C-31-M-12-Edge_Silkscreen_Removed -> easyeda2kicad:USB_C_Receptacle_HRO_TYPE-C-31-M-12-Edge_Silkscreen_Removed
- U12: footprint amemb-Package_LGA:amemb-ADXL367_LGA-12_2.11x2.21mm_P0.5mm_LayoutBorder2x4y -> easyeda2kicad:ADXL367_LGA-12_2.11x2.21mm_P0.5mm_LayoutBorder2x4y
- U9: footprint amemb-Conenctor_JST:JST_SH_SM04B-SRSS-TB_1x04-1MP_P1.00mm_Horizontal -> easyeda2kicad:JST_SH_SM04B-SRSS-TB_1x04-1MP_P1.00mm_Horizontal
Changed lines of the file:
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@@
 				(loss_tangent 0.02)
 			)
-			(layer "In2.Cu"
+			(layer "In1.Cu"
 				(type "copper")
 				(thickness 0.035)
@@
 				(loss_tangent 0.02)
 			)
-			(layer "In3.Cu"
+			(layer "In1.Cu"
 				(type "copper")
 				(thickness 0.035)
@@
 		(property "LCSC" "C49307573"
 			(at 0 0 0)
+			(unlocked yes)
 			(layer "F.Fab")
 			(hide yes)
 			(effects
 				(font
-					(size 1.27 1.27)
+					(size 1 1)
 					(thickness 0.15)
 				)
@@
 		(fp_poly
 			(pts
-				(xy -0.3375 -0.600001) (xy -0.2375 -0.75) (xy -0.4375 -0.75)
+				(xy -0.3375 -0.6) (xy -0.2375 -0.75) (xy -0.4375 -0.75)
 			)
 			(stroke
@@
 			(layer "F.SilkS")
 		)
-		(fp_poly
-			(pts
-				(xy -0.7 -0.7) (xy 0.7 -0.7) (xy 0.7 0.7) (xy -0.7 0.7)
-			)
+		(fp_rect
+			(start -0.7 -0.7)
+			(end 0.7 0.7)
 			(stroke
 				(width 0.05)
@@
 			)
 		)
-		(property "LCSC" "C965807"
+		(property "LCSC" "C7496819"
 			(at 0 0 0)
 			(layer "F.Fab")
@@
 		)
 	)
-	(footprint "amemb-Connector_USB:USB_C_Receptacle_HRO_TYPE-C-31-M-12-Edge_Silkscreen_Removed"
+	(footprint "easyeda2kicad:USB_C_Receptacle_HRO_TYPE-C-31-M-12-Edge_Silkscreen_Removed"
 		(layer "F.Cu")
 		(at 101.79376 66.7212 -90)
@@
 			)
 		)
-		(property "LCSC" "C5217869"
+		(property "LCSC Part" "C5217869"
 			(at 0 0 0)
 			(layer "F.Fab")
@@
 			)
 		)
-		(property "LCSC Part" "C5217869"
+		(property "LCSC" "C5217869"
 			(at 0 0 0)
+			(unlocked yes)
 			(layer "F.Fab")
 			(hide yes)
 			(effects
 				(font
-					(size 1.27 1.27)
+					(size 1 1)
 					(thickness 0.15)
 				)
@@
 			)
 		)
-		(property "LCSC" "C965807"
+		(property "LCSC" "C7496819"
 			(at 0 0 0)
 			(layer "F.Fab")
@@
 		)
 	)
-	(footprint "amemb-Package_LGA:amemb-ADXL367_LGA-12_2.11x2.21mm_P0.5mm_LayoutBorder2x4y"
+	(footprint "easyeda2kicad:ADXL367_LGA-12_2.11x2.21mm_P0.5mm_LayoutBorder2x4y"
 		(layer "F.Cu")
 		(at 127.73016 77.22598 180)
@@
 		(tags "ADI LGA NoLead")
 		(property "Reference" "U12"
-			(at 0 -1.95 0)
+			(at 0 -1.95 180)
 			(layer "F.SilkS")
 			(hide yes)
@@
 		)
 		(property "Value" "ADXL367"
-			(at 0 1.95 0)
+			(at 0 1.95 180)
 			(layer "F.Fab")
 			(effects
@@
 		)
 		(property "Datasheet" ""
-			(at 0 0 0)
+			(at 0 0 180)
 			(layer "F.Fab")
 			(hide yes)
@@
 		)
 		(property "Description" ""
-			(at 0 0 0)
+			(at 0 0 180)
 			(layer "F.Fab")
 			(hide yes)
@@
 		)
 		(property "LCSC" "C17643415"
-			(at 0 0 0)
+			(at 0 0 180)
 			(layer "F.Fab")
 			(hide yes)
@@
 		)
 		(fp_text user "${REFERENCE}"
-			(at 0 0 90)
+			(at 0 0 270)
 			(layer "F.Fab")
 			(effects
@@
 		)
 		(pad "1" smd roundrect
-			(at -0.86 -0.75 180)
+			(at -0.86 -0.75)
 			(size 0.39 0.33)
 			(layers "F.Cu" "F.Mask" "F.Paste")
@@
 		)
 		(pad "2" smd roundrect
-			(at -0.86 -0.25 180)
+			(at -0.86 -0.25)
 			(size 0.39 0.33)
 			(layers "F.Cu" "F.Mask" "F.Paste")
@@
 		)
 		(pad "3" smd roundrect
-			(at -0.86 0.25 180)
+			(at -0.86 0.25)
 			(size 0.39 0.33)
 			(layers "F.Cu" "F.Mask" "F.Paste")
@@
 		)
 		(pad "4" smd roundrect
-			(at -0.86 0.75 180)
+			(at -0.86 0.75)
 			(size 0.39 0.33)
 			(layers "F.Cu" "F.Mask" "F.Paste")
@@
 		)
 		(pad "5" smd roundrect
-			(at -0.25 0.91 180)
+			(at -0.25 0.91)
 			(size 0.33 0.39)
 			(layers "F.Cu" "F.Mask" "F.Paste")
@@
 		)
 		(pad "6" smd roundrect
-			(at 0.25 0.91 180)
+			(at 0.25 0.91)
 			(size 0.33 0.39)
 			(layers "F.Cu" "F.Mask" "F.Paste")
@@
 		)
 		(pad "7" smd roundrect
-			(at 0.86 0.75 180)
+			(at 0.86 0.75)
 			(size 0.39 0.33)
 			(layers "F.Cu" "F.Mask" "F.Paste")
@@
 		)
 		(pad "8" smd roundrect
-			(at 0.86 0.25 180)
+			(at 0.86 0.25)
 			(size 0.39 0.33)
 			(layers "F.Cu" "F.Mask" "F.Paste")
@@
 		)
 		(pad "9" smd roundrect
-			(at 0.86 -0.25 180)
+			(at 0.86 -0.25)
 			(size 0.39 0.33)
 			(layers "F.Cu" "F.Mask" "F.Paste")
@@
 		)
 		(pad "10" smd roundrect
-			(at 0.86 -0.75 180)
+			(at 0.86 -0.75)
 			(size 0.39 0.33)
 			(layers "F.Cu" "F.Mask" "F.Paste")
@@
 		)
 		(pad "11" smd roundrect
-			(at 0.25 -0.91 180)
+			(at 0.25 -0.91)
 			(size 0.33 0.39)
 			(layers "F.Cu" "F.Mask" "F.Paste")
@@
 		)
 		(pad "12" smd roundrect
-			(at -0.25 -0.91 180)
+			(at -0.25 -0.91)
 			(size 0.33 0.39)
 			(layers "F.Cu" "F.Mask" "F.Paste")
@@
 		)
 		(embedded_fonts no)
-		(model "${KICAD10_3DMODEL_DIR}/amemb-Package_LGA.3dshapes/amemb-ADXL367_LGA-12_2.11x2.21mm_P0.5mm_LayoutBorder2x4y.step"
-			(offset
-				(xyz 0 0 0)
-			)
-			(scale
-				(xyz 1 1 1)
-			)
-			(rotate
-				(xyz 0 0 0)
-			)
-		)
 	)
 	(footprint "passives:C_0201_0603Metric_L"
@@
 			)
 		)
-		(property "LCSC" "C5217875"
+		(property "LCSC Part" "C5217875"
 			(at 0 0 0)
 			(layer "F.Fab")
@@
 			)
 		)
-		(property "LCSC Part" "C5217875"
+		(property "LCSC" "C5217875"
 			(at 0 0 0)
+			(unlocked yes)
 			(layer "F.Fab")
 			(hide yes)
 			(effects
 				(font
-					(size 1.27 1.27)
+					(size 1 1)
 					(thickness 0.15)
 				)
@@
 		(duplicate_pad_numbers_are_jumpers no)
 		(fp_line
-			(start -0.89 1.089999)
+			(start -0.89 1.09)
 			(end -0.89 1.14)
 			(stroke
@@
 		)
 		(fp_line
-			(start -0.82 -1.190001)
+			(start -0.82 -1.19)
 			(end -0.25 -1.19)
 			(stroke
@@
 		(fp_line
 			(start -0.82 -1.14)
-			(end -0.82 -1.190001)
+			(end -0.82 -1.19)
 			(stroke
 				(width 0.15)
@@
 		(fp_line
 			(start 0.89 1.14)
-			(end 0.89 1.089999)
+			(end 0.89 1.09)
 			(stroke
 				(width 0.15)
@@
 			(layer "F.SilkS")
 		)
-		(fp_poly
-			(pts
-				(xy -1.2 -1.35) (xy 1.2 -1.35) (xy 1.2 1.35) (xy -1.2 1.35)
-			)
+		(fp_rect
+			(start -1.2 -1.35)
+			(end 1.2 1.35)
 			(stroke
 				(width 0.05)
@@
 		)
 		(pad "5" smd roundrect
-			(at -0.74 0.799999 270)
+			(at -0.74 0.8 270)
 			(size 0.2 0.825)
 			(layers "F.Cu" "F.Mask" "F.Paste")
@@
 		)
 		(pad "7" smd roundrect
-			(at 0.74 0.799999 270)
+			(at 0.74 0.8 270)
 			(size 0.2 0.825)
 			(layers "F.Cu" "F.Mask" "F.Paste")
@@
 		)
 		(pad "11" smd roundrect
-			(at 0.74 -0.799999 270)
+			(at 0.74 -0.8 270)
 			(size 0.2 0.825)
 			(layers "F.Cu" "F.Mask" "F.Paste")
@@
 		)
 	)
-	(footprint "amemb-Conenctor_JST:JST_SH_SM04B-SRSS-TB_1x04-1MP_P1.00mm_Horizontal"
+	(footprint "easyeda2kicad:JST_SH_SM04B-SRSS-TB_1x04-1MP_P1.00mm_Horizontal"
 		(layer "F.Cu")
 		(at 108.72016 52.7212 180)
@@
 		)
 		(embedded_fonts no)
-		(model "${KICAD9_3DMODEL_DIR}/Connector_JST.3dshapes/JST_SH_SM04B-SRSS-TB_1x04-1MP_P1.00mm_Horizontal.step"
+		(model "${KICAD10_3DMODEL_DIR}/Connector_JST.3dshapes/JST_SH_SM04B-SRSS-TB_1x04-1MP_P1.00mm_Horizontal.step"
 			(offset
 				(xyz 0 0 0)
@@
 	)
 	(group "USB-C Receptacle with ESD + 1A fuse"
-		(lib_id "amemb-USB:USB-C Receptacle with ESD + 1A fuse")
+		(lib_id "Sidewalk_Devkit:USB-C Receptacle with ESD + 1A fuse")
 		(members "58438c4b-0903-431d-9726-18c6e11de30c" "cbf1d1c7-6b73-428d-93eb-569b9c591332")
 	)
 	(group "SX1262 IPD, 915MHz"
-		(lib_id "amemb-RF:SX1262 IPD, 915MHz")
+		(lib_id "Sidewalk_Devkit:SX1262 IPD, 915MHz")
 		(members "02363cec-b62e-4482-8401-e0d71b1aa7d7" "06bf074b-7a48-4acd-8cfe-6369399424bc"
 			"22a25d17-2ce7-4552-afc5-34a9b796fd4f" "2d260dcc-2968-4b9d-bb21-f4ddf6553dd3"
@@
 		)
 	)
+	(group "nRF52833 Debugger"
+		(lib_id "Sidewalk_Devkit:nRF52833 Debugger")
+		(members "146a8da8-f61c-451a-8f55-30583c748b01" "1de7708b-bd4c-464d-adfd-2804f0be6844"
+			"2df902f3-2513-40ab-a0ab-cdbf8b42c949" "31cc088b-a96b-4c5b-a76b-b16a0aadc326"
+			"37a58488-c04b-4ae9-b2a8-fdbb4a9ba803" "447861d9-7bd4-40a3-b985-f18c008f0f3a"
+			"598d7d23-c09a-47c4-a70a-aa72c971abc5" "5ad5da3e-21d7-4edb-935c-930dfa6d0e82"
+			"5e19ec01-1bba-4684-aedf-4d9ad2b50487" "6815ad2b-dcdb-43bb-9744-4a80ed8d4e79"
+			"689ba9ab-d215-4db6-b777-eb3f419c12b7" "6c2ba084-363e-451f-8f84-5c3e1a27a5b2"
+			"6cda3223-3991-48d8-aa1c-2f8b5a4fa660" "768dfc5b-cc90-43ce-9b79-baa78ab2d197"
+			"8e23d461-3422-4e5f-90f9-0e15a6e566c0" "9438a66c-1d8c-47f4-8c4d-a2ba64232b95"
+			"95d9f842-13d1-4cb3-b26a-4486ee3175cd" "9c1cfee1-1048-4072-9282-d01215c1c9e2"
+			"b2fda719-0716-4421-a6da-fff562f899a0" "bb362900-2c98-4027-8b48-1dfd49795cfb"
+			"bc024651-ab41-41f1-8d52-9fc25a5dee78" "bc4bc5a3-67ba-4616-b874-92ec7b6c37a6"
+			"c4722501-31aa-4e0a-82aa-f1d45ebaf430" "cad0626c-77d7-4b86-80ec-2dcb0bdf4572"
+			"d69edab0-2a61-43e2-9597-f19c28fbffef" "d7917d72-c433-4a49-817c-736d20ad5cd5"
+			"ddfb2c45-30cf-4f02-b0cc-7135e5fa0726" "e1526fa4-3386-400b-8a44-9c160bdf2b52"
+			"f7fe470c-5fdd-4b30-8e4a-bbd31f0d4e3c" "f9c4303e-cf87-4f00-867d-76f1ff354f26"
+			"fad087a7-a12d-4b60-886b-af81f70d1959"
+		)
+	)
 	(group "nRF54L15-QFXX_Reference_Design"
 		(lib_id "nRF54L:nRF54L15-QFXX_Reference_Design")
@@
 	)
 	(group "SX1262 IPD, 915MHz"
-		(lib_id "amemb-RF:SX1262 IPD, 915MHz")
+		(lib_id "Sidewalk_Devkit:SX1262 IPD, 915MHz")
 		(members "0036f37e-a364-4fe9-9b21-da86c1a9bd6c" "0543493a-a913-4e05-acb6-cd00772528f6"
 			"05b11da2-aea2-45a5-9daa-dec2a7ded3a1" "0cfba180-4165-4f58-aba8-986fd5c54533"

Commit message: Added external current measurement for L15 and SX1262
Parts:
- added C60: 1uF, passives:C_0201_0603Metric_L, F.Cu at (121.3, 52.8)
- added C61: 1uF, passives:C_0201_0603Metric_L, F.Cu at (122.9, 52.8)
- added C62: 1uF, passives:C_0201_0603Metric_L, F.Cu at (121.3, 50.7)
- added C63: 1uF, passives:C_0201_0603Metric_L, F.Cu at (122.9, 50.7)
- added C64: 1uF, passives:C_0201_0603Metric_L, F.Cu at (135.6, 50.7)
- added C65: 1uF, passives:C_0201_0603Metric_L, F.Cu at (137.2, 50.7)
- added C66: 1uF, passives:C_0201_0603Metric_L, F.Cu at (137.2, 52.7)
- added C67: 1uF, passives:C_0201_0603Metric_L, F.Cu at (135.6, 52.8)
- added J5: Conn_01x03_Pin, Connector_PinHeader_2.54mm:PinHeader_1x03_P2.54mm_Vertical, F.Cu at (125.8, 51.7)
- added J6: Conn_01x03_Pin, Connector_PinHeader_2.54mm:PinHeader_1x03_P2.54mm_Vertical, F.Cu at (139.8, 51.7)
- added Q2: Q_NMOS_GSD, Package_DFN_QFN:Diodes_DFN1006-3, F.Cu at (119.7, 51.8)
- added Q3: Q_NMOS_GSD, Package_DFN_QFN:Diodes_DFN1006-3, F.Cu at (134.0, 51.7)
- added R14: 100kR, passives:C_0201_0603Metric_L, F.Cu at (119.7, 50.6)
- added R15: 100kR, passives:C_0201_0603Metric_L, F.Cu at (119.7, 52.9)
- added R16: 100kR, passives:C_0201_0603Metric_L, F.Cu at (134.0, 50.6)
- added R18: 100kR, passives:C_0201_0603Metric_L, F.Cu at (134.0, 52.8)
- added TP36: TestPoint, TestPoint:TestPoint_Pad_D1.0mm, B.Cu at (112.1, 52.5)
- added TP37: TestPoint, TestPoint:TestPoint_Pad_D1.0mm, B.Cu at (117.5, 52.3)
- added TP38: TestPoint, TestPoint:TestPoint_Pad_D1.0mm, B.Cu at (140.6, 55.1)
- added U14: TPS22991, easyeda2kicad:4-UQFN-0.9x0.8mm, F.Cu at (121.3, 51.8)
- added U15: TPS22991, easyeda2kicad:4-UQFN-0.9x0.8mm, F.Cu at (122.9, 51.8)
- added U16: TPS22991, easyeda2kicad:4-UQFN-0.9x0.8mm, F.Cu at (135.6, 51.7)
- added U17: TPS22991, easyeda2kicad:4-UQFN-0.9x0.8mm, F.Cu at (137.2, 51.7)
- moved TP7 5.61 mm to (120.9, 54.4)
Connections:
- C22 pad 1: VDD_SX1262 -> Net-(U16-VIN)
- C24 pad 1: VDD_nRF -> Net-(U14-VIN)
- L5 pad 1: VDD_nRF -> Net-(U14-VIN)
- L6 pad 2: VDD_SX1262 -> Net-(U16-VIN)
- TP7 pad 1: VDD_nRF -> Net-(U14-VIN)
- TP8 pad 1: VDD_SX1262 -> Net-(U16-VIN)
- U2 pad 1: VDD_nRF -> Net-(U14-VIN)
- U2 pad 32: VDD_SX1262 -> Net-(U16-VIN)
- U7 pad 6: unconnected-(U7-P1.09-Pad6) -> /Debugger/EXT_PWR
Routing:
- net /Debugger/EXT_PWR: track 0.00 -> 60.2 mm, vias 0 -> 5
- net Net-(U14-VIN): track 0.00 -> 31.3 mm, vias 0 -> 6
- net Net-(U16-VIN): track 0.00 -> 25.7 mm, vias 0 -> 2
- net VDD_nRF: track 77.4 -> 100.6 mm, vias 11 -> 12
- net Net-(Q3-D): track 0.00 -> 11.4 mm, vias 0 -> 2
- net Net-(Q2-D): track 0.00 -> 6.84 mm, vias 0 -> 2
- net Net-(J6-Pin_1): track 0.00 -> 5.08 mm, vias 0 -> 1
- net VDD_SX1262: track 33.4 -> 28.4 mm, vias 5 -> 2
- net Net-(J5-Pin_1): track 0.00 -> 5.01 mm, vias 0 -> 1
- net GND: track 73.2 -> 76.5 mm, vias 134 -> 145
- net /BUTTON0: track 94.8 -> 96.5 mm, vias 1 -> 3
- net Net-(J3-SWCLK): track 13.4 -> 12.8 mm
- net Net-(U2-SW1): track 4.35 -> 3.72 mm
- net /nPM1300/SDA: track 44.9 -> 44.6 mm, vias 2 -> 3
- net /nPM1300/SCL: track 45.8 -> 45.7 mm, vias 2 -> 3
- added copper zone on In3.Cu, net GND
- added copper zone on In4.Cu, net GND
- added copper zone on F.Cu, net Net-(U14-VIN)
- added copper zone on F.Cu, net Net-(U16-VIN)
- removed copper zone on F.Cu, net VDD_nRF
Other:
- board text added: "GND"
- board text added: "IDD"
- board text added: "Rev: ${REVISION} @{vcsidentifier(8)}@{vcsdirtysuffix()}"
- board text added: "nRF54L"
- board text removed: "Rev: ${REVISION} @{vcsidentifier(8)} @{vcsdirtysuffix()}"
