File: Sidewalk_Devkit.kicad_pcb (KiCad board)
At the start: 6 copper layers, 55 x 34 mm, 183 parts, among them J1 USB_C_Receptacle_USB2.0_16P, J2 Conn_Coaxial_Small, J3 Conn_ARM_SWD_TagConnect_TC203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, J4 Conn_01x02_MountingPin, J5 Conn_01x03_Pin, J6 Conn_01x03_Pin, J7 Conn_01x05_MountingPin, Q1 Q_NMOS_GSD, Q2 Q_NMOS_GSD, Q3 Q_NMOS_GSD, SW1 SW_Push, SW2 SW_Push, U1 nRF54L15-QFAA, U10 TPS22991, U11 SHT4x, U12 ADXL367, U13 ZD25WQ16CEIGR, U14 TPS22991, U15 TPS22991, U16 TPS22991, U17 TPS22991, U2 nPM1300-QEAA, U3 SX1262IMLTRT, U4 BGS12WN6E6327, U5 USBLC6-2P6, U6 TXU0204RUTR, U7 nRF52833-QDXX, U8 TXU0101DRYR, U9 STEMMA-QT, X1 32MHz, X2 32.768kHz, Y1 32MHz, 10pF, Y2 32MHz, 10pF

Commit message: Revision 0.2
Parts:
- added U18: LIS2DH, Package_LGA:LGA-14_2x2mm_P0.35mm_LayoutBorder3x4y, F.Cu at (127.3, 77.7)
- C52, C53: value 300pF -> 330pF
- C56: value 220nF -> 1uF
- U12: value ADXL367 -> TMUX1511RSVR; footprint easyeda2kicad:ADXL367_LGA-12_2.11x2.21mm_P0.5mm_LayoutBorder2x4y -> easyeda2kicad:UTQFN-16_L2.6-W1.8-P0.40-BL
- U13: value ZD25WQ16CEIGR -> W25Q16JVUXIQ
- U4: value BGS12WN6E6327 -> BGS12SN6E6327XTSA1
- moved C56 6.75 mm to (128.7, 71.3), turned to 0 degrees
- moved U12 4.61 mm to (127.2, 72.7)
- moved C50 3.95 mm to (123.6, 68.0)
- moved C36 3.95 mm to (117.5, 75.0)
- moved C37 3.95 mm to (118.0, 75.0)
- moved C42 3.95 mm to (120.4, 74.1)
- moved C45 3.95 mm to (120.5, 77.2)
- moved TP32 3.95 mm to (114.4, 68.3)
- moved U8 3.95 mm to (123.6, 69.3)
- moved Y2 3.95 mm to (118.8, 77.2)
- moved C35 3.95 mm to (113.7, 69.0)
- moved C38 3.95 mm to (120.4, 68.0)
- moved C39 3.95 mm to (115.6, 67.3)
- moved C40 3.95 mm to (113.7, 72.1)
- moved C41 3.95 mm to (116.6, 67.0)
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Connections:
- AE1 pad 1: unconnected-(AE1-FEED-Pad1) -> Net-(AE1-FEED)
- AE1 pad 2: Net-(AE1-PCB_Trace) -> unconnected-(AE1-PCB_Trace-Pad2)
- C56 pad 1: Net-(U12-V_{REG_OUT}) -> /Debugger/LEVEL_SHIFT_VDD
- U12 pad 1: GND -> /Debugger/LEVEL_SHIFT_VDD
- U12 pad 10: SENSOR_VDD -> /Debugger/TX
- U12 pad 11: GND -> /Debugger/LEVEL_SHIFT_VDD
- U12 pad 12: SENSOR_VDD -> unconnected-(U12-N.C.-Pad12)
- U12 pad 2: /nRF54L15/SDA_SENSOR -> /Debugger/TARGET_SWDCLK
- U12 pad 3: GND -> /Debugger/INT_TRG.SWDCLK
- U12 pad 4: /nRF54L15/SCL_SENSOR -> /Debugger/LEVEL_SHIFT_VDD
- U12 pad 5: /nRF54L15/INT1 -> /Debugger/RX
- U12 pad 6: unconnected-(U12-INT2-Pad6) -> /Debugger/INT_TRG.RX
- U12 pad 7: GND -> unconnected-(U12-N.C.-Pad7)
- U12 pad 8: unconnected-(U12-ADC_{IN}-Pad8) -> GND
- U12 pad 9: Net-(U12-V_{REG_OUT}) -> /Debugger/INT_TRG.TX
- U6 pad 10: /Debugger/TARGET_SWDCLK -> /Debugger/INT_TRG.SWDCLK
- U6 pad 7: /Debugger/TARGET_SWDIO -> /Debugger/INT_TRG.SWDIO
- U6 pad 8: /Debugger/TX -> /Debugger/INT_TRG.TX
- U6 pad 9: /Debugger/RX -> /Debugger/INT_TRG.RX
- U8 pad 4: /Debugger/TARGET_SWDIO -> /Debugger/INT_TRG.SWDIO
- Z5 pad 2: Net-(AE1-PCB_Trace) -> Net-(AE1-FEED)
- Z6 pad 2: Net-(AE1-PCB_Trace) -> Net-(AE1-FEED)
Routing:
- net /nPM1300/nPM1300.INT: track 77.3 -> 45.2 mm
- net /nRF54L15/SDA_STEMMA: track 62.4 -> 46.1 mm
- net /Debugger/INT_TRG.SWDIO: track 0.00 -> 15.8 mm, vias 0 -> 2
- net /Debugger/LEVEL_SHIFT_VDD: track 9.48 -> 23.3 mm
- net SENSOR_VDD: track 37.3 -> 46.9 mm
- net /Debugger/EXT_PWR: track 60.2 -> 53.2 mm, vias 5 -> 6
- net /Debugger/TARGET_SWDIO: track 42.2 -> 36.1 mm, vias 4 -> 3
- net /Debugger/TARGET_SWDCLK: track 47.5 -> 41.9 mm
- net /Debugger/INT_TRG.TX: track 0.00 -> 5.18 mm
- net /Debugger/INT_TRG.SWDCLK: track 0.00 -> 4.51 mm
- net VDD_nRF: track 100.6 -> 97.2 mm, vias 12 -> 13
- net /nRF54L15/SCL_SENSOR: track 18.9 -> 22.2 mm, vias 2 -> 4
- net Net-(AE1-PCB_Trace): track 3.22 -> 0.00 mm
- net Net-(AE1-FEED): track 0.00 -> 3.22 mm
- net GND: track 76.5 -> 79.5 mm, vias 145 -> 149
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Other:
- board text removed: "DEBUGGER"
