File: Sidewalk_Devkit.kicad_pcb (KiCad board)
At the start: 6 copper layers, 55 x 34 mm, 184 parts, among them J1 USB_C_Receptacle_USB2.0_16P, J2 Conn_Coaxial_Small, J3 Conn_ARM_SWD_TagConnect_TC203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, J4 Conn_01x02_MountingPin, J5 Conn_01x03_Pin, J6 Conn_01x03_Pin, J7 Conn_01x05_MountingPin, Q1 Q_NMOS_GSD, Q2 Q_NMOS_GSD, Q3 Q_NMOS_GSD, SW1 SW_Push, SW2 SW_Push, U1 nRF54L15-QFAA, U10 TPS22991, U11 SHT4x, U12 TMUX1511RSVR, U13 W25Q16JVUXIQ, U14 TPS22991, U15 TPS22991, U16 TPS22991, U17 TPS22991, U18 LIS2DH, U2 nPM1300-QEAA, U3 SX1262IMLTRT, U4 BGS12SN6E6327XTSA1, U5 USBLC6-2P6, U6 TXU0204RUTR, U7 nRF52833-QDXX, U8 TXU0101DRYR, U9 STEMMA-QT, X1 32MHz, X2 32.768kHz, Y1 32MHz, 10pF, Y2 32MHz, 10pF

Commit message: Updates for V2
Parts:
- U13: value W25Q16JVUXIQ -> MX25R1635FZUIL0
- X1: value 32MHz -> 32MHz, 10pF
